Commit message: ステアリングを位置指定・速度制御にした

File: urdf/steering/steering.urdf.xacro (robot description, xacro)
@@ -11,4 +11,5 @@
       <child link="${prefix}_steering_link"/>
       <insert_block name="joint_axis"/>
+      <limit effort="10" velocity="25"/>
     </joint>
     <link name="${prefix}_steering_link">
@@ -42,8 +43,8 @@
       <type>transmission_interface/SimpleTransmission</type>
       <joint name="${prefix}_steering_joint">
-        <hardwareInterface>hardware_interface/PositionJointInterface</hardwareInterface>
+        <hardwareInterface>hardware_interface/VelocityJointInterface</hardwareInterface>
       </joint>
       <actuator name="${prefix}_steering_motor">
-        <hardwareInterface>hardware_interface/PositionJointInterface</hardwareInterface>
+        <hardwareInterface>hardware_interface/velocityJointInterface</hardwareInterface>
         <mechanicalReduction>30</mechanicalReduction>
       </actuator>

Commit message: 全ジョイントを動かせるようにした

File: urdf/steering/steering.urdf.xacro (robot description, xacro)
@@ -11,5 +11,5 @@
       <child link="${prefix}_steering_link"/>
       <insert_block name="joint_axis"/>
-      <limit effort="10" velocity="25"/>
+      <limit effort="30" velocity="25"/>
     </joint>
     <link name="${prefix}_steering_link">

File: urdf/wheel/wheel.urdf.xacro (robot description, xacro)
@@ -11,4 +11,5 @@
       <child link="${prefix}_wheel_link"/>
       <insert_block name="joint_axis"/>
+      <limit velocity="25" effort="30"/>
     </joint>
     <link name="${prefix}_wheel_link">

Commit message: ステアリングをrevoluteに変更.また,ゲインを変更

File: urdf/steering/steering.urdf.xacro (robot description, xacro)
@@ -6,10 +6,10 @@
   <property name="steering_mass" value="5.0"/>
   <xacro:macro name="steering" params="prefix parent *joint_origin *joint_axis">
-    <joint name="${prefix}_steering_joint" type="continuous">
+    <joint name="${prefix}_steering_joint" type="revolute">
       <insert_block name="joint_origin"/>
       <parent link="${parent}"/>
       <child link="${prefix}_steering_link"/>
       <insert_block name="joint_axis"/>
-      <limit effort="30" velocity="25"/>
+      <limit effort="30" velocity="25" upper="${M_PI/1.5}" lower="${-M_PI/1.5}"/>
     </joint>
     <link name="${prefix}_steering_link">
