Commit message: ステアリングを追加

File: urdf/base/base.urdf.xacro (robot description, xacro)
@@ -10,5 +10,5 @@
     <link name="base_link">
       <visual>
-        <origin xyz="0 0 0.5" rpy="0 0 0"/>
+        <origin xyz="0 0 0.25" rpy="0 0 0"/>
         <geometry>
           <box size="0.5 0.5 0.5"/>

Commit message: 胴体のみstlに置き換えた

File: urdf/base/base.urdf.xacro (robot description, xacro)
@@ -10,18 +10,20 @@
     <link name="base_link">
       <visual>
-        <origin xyz="0 0 0.25" rpy="0 0 0"/>
+        <origin xyz="0.200 -0.630 0.060" rpy="${M_PI/2} 0 ${M_PI/2}"/>
         <geometry>
-          <box size="0.5 0.5 0.5"/>
+          <mesh filename="package://mygazebo/meshes/STL/base.stl" scale="0.001 0.001 0.001"/>
         </geometry>
       </visual>
       <collision>
-        <origin xyz="0 0 0.5" rpy="0 0 0"/>
+        <origin xyz="0.200 -0.630 0.060" rpy="${M_PI/2} 0 ${M_PI/2}"/>
         <geometry>
-          <box size="0.5 0.5 0.5"/>
+          <mesh filename="package://mygazebo/meshes/STL/base.stl" scale="0.001 0.001 0.001"/>
         </geometry>
       </collision>
       <inertial>
-        <origin xyz="0 0 0.5" rpy="0 0 0"/>
+        <origin xyz="0.200 -0.630 0.060" rpy="${M_PI/2} 0 ${M_PI/2}"/>
         <box_inertial mass="5.0" height="0.5" width="0.5" depth="0.5"/>
+        <mass value="43.24"/>
+        <inertia ixx="4.115" ixy="0" ixz="0" iyz="0" iyy="4.207" izz="4.076"/>
       </inertial>
     </link>
