Commit message: パッケージ構成を変更

File: four_wheel_drive_independent_steering/urdf/base/base.urdf.xacro (robot description, xacro)
@@ -1,5 +1,5 @@
 <?xml version="1.0"?>
 <robot xmlns:xacro="http://ros.org/wiki/xacro">
-  <xacro:include filename="$(find mygazebo)/urdf/common.xacro"/>
+  <xacro:include filename="$(find four_wheel_drive_independent_steering)/urdf/common.xacro"/>
   <xacro:macro name="base" params="parent *joint_origin">
     <joint name="base_link_joint" type="fixed">
@@ -12,5 +12,5 @@
         <origin xyz="0.200 -0.630 0.060" rpy="${M_PI/2} 0 ${M_PI/2}"/>
         <geometry>
-          <mesh filename="package://mygazebo/meshes/STL/base.stl" scale="0.001 0.001 0.001"/>
+          <mesh filename="package://four_wheel_drive_independent_steering/meshes/STL/base.stl" scale="0.001 0.001 0.001"/>
         </geometry>
       </visual>
@@ -18,5 +18,5 @@
         <origin xyz="0.200 -0.630 0.060" rpy="${M_PI/2} 0 ${M_PI/2}"/>
         <geometry>
-          <mesh filename="package://mygazebo/meshes/STL/base.stl" scale="0.001 0.001 0.001"/>
+          <mesh filename="package://four_wheel_drive_independent_steering/meshes/STL/base.stl" scale="0.001 0.001 0.001"/>
         </geometry>
       </collision>

File: four_wheel_drive_independent_steering/urdf/steering/steering.urdf.xacro (robot description, xacro)
@@ -1,5 +1,5 @@
 <?xml version="1.0"?>
 <robot xmlns:xacro="http://ros.org/wiki/xacro">
-  <xacro:include filename="$(find mygazebo)/urdf/common.xacro"/>
+  <xacro:include filename="$(find four_wheel_drive_independent_steering)/urdf/common.xacro"/>
   <property name="steering_radius" value="0.100"/>
   <property name="steering_width" value="0.100"/>

File: four_wheel_drive_independent_steering/urdf/wheel/wheel.urdf.xacro (robot description, xacro)
@@ -1,5 +1,5 @@
 <?xml version="1.0"?>
 <robot xmlns:xacro="http://ros.org/wiki/xacro">
-  <xacro:include filename="$(find mygazebo)/urdf/common.xacro"/>
+  <xacro:include filename="$(find four_wheel_drive_independent_steering)/urdf/common.xacro"/>
   <property name="wheel_radius" value="0.075"/>
   <property name="wheel_width" value="0.030"/>
