Commit message: パラメータ調整

File: four_wheel_drive_independent_steering/urdf/steering/steering.urdf.xacro (robot description, xacro)
@@ -11,5 +11,5 @@
       <child link="${prefix}_steering_link"/>
       <insert_block name="joint_axis"/>
-      <limit effort="30" velocity="25" upper="${M_PI/1.5}" lower="${-M_PI/1.5}"/>
+      <limit effort="30" velocity="30" upper="${M_PI/1.5}" lower="${-M_PI/1.5}"/>
     </joint>
     <link name="${prefix}_steering_link">

File: four_wheel_drive_independent_steering/urdf/wheel/wheel.urdf.xacro (robot description, xacro)
@@ -11,5 +11,5 @@
       <child link="${prefix}_wheel_link"/>
       <insert_block name="joint_axis"/>
-      <limit velocity="25" effort="30"/>
+      <limit velocity="30" effort="30"/>
     </joint>
     <link name="${prefix}_wheel_link">

Commit message: パラメータ変更

File: four_wheel_drive_independent_steering/urdf/steering/steering.urdf.xacro (robot description, xacro)
@@ -11,5 +11,5 @@
       <child link="${prefix}_steering_link"/>
       <insert_block name="joint_axis"/>
-      <limit effort="30" velocity="30" upper="${M_PI/1.5}" lower="${-M_PI/1.5}"/>
+      <limit effort="2.323" velocity="30" upper="${M_PI/1.5}" lower="${-M_PI/1.5}"/>
     </joint>
     <link name="${prefix}_steering_link">

File: four_wheel_drive_independent_steering/urdf/wheel/wheel.urdf.xacro (robot description, xacro)
@@ -11,5 +11,5 @@
       <child link="${prefix}_wheel_link"/>
       <insert_block name="joint_axis"/>
-      <limit velocity="30" effort="30"/>
+      <limit velocity="30" effort="2.323"/>
     </joint>
     <link name="${prefix}_wheel_link">
